File: PCB/can.kicad_sch (KiCad schematic)
At the start: 9 parts, among them J3 CAN, U6 MCP2562-E-SN

Commit message: Generate project from template
Other:
- title: template_pretty_name -> NAUTILUS Bms Test Board
Changed lines of the file:
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@@
 	(paper "A4")
 	(title_block
-		(title "template_pretty_name")
+		(title "NAUTILUS Bms Test Board")
 	)
 	(text "ESD\nprotection"
