File: PCB/mcu.kicad_sch (KiCad schematic)
At the start: 35 parts, among them J1 STDC-14 Debug, Q1 2N7002, SW1 Reset, U1 ADM1818, U2 W25N512GVEIG, U3 STM32G473RCTx, Y1 16MHz/8pF

Commit message: Generate project from template
Other:
- title: template_pretty_name -> NAUTILUS Bms Test Board
Changed lines of the file:
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@@
 	(paper "A4")
 	(title_block
-		(title "template_pretty_name")
+		(title "NAUTILUS Bms Test Board")
 	)
 	(text "512Mb NAND Flash"
