File: PCB/nautilus-bms-test-PCB.kicad_sch (KiCad schematic)
At the start: 0 parts

Commit message: Generate project from template
Other:
- title: template_pretty_name -> NAUTILUS Bms Test Board
Changed lines of the file:
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@@
 	(paper "A4")
 	(title_block
-		(title "template_pretty_name")
+		(title "NAUTILUS Bms Test Board")
 	)
 	(no_connect
