File: PCB/stack_format.kicad_sch (KiCad schematic)
At the start: 9 parts, among them J5 EdgeConn_FC

Commit message: Generate project from template
Other:
- title: template_pretty_name -> NAUTILUS Bms Test Board
Changed lines of the file:
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@@
 	(paper "A4")
 	(title_block
-		(title "template_pretty_name")
+		(title "NAUTILUS Bms Test Board")
 	)
 	(junction
